Commit message: changed 'package' to 'model'

File: pibot_description/models/iti0201_robot_cone/urdf/pibot.urdf (robot description, URDF)
Before this commit: robot pibot, 28 links, 27 joints
Links:
- link base_with_casters: geometry collision mesh filename=model://iti0201_robot/meshes/base_green.dae; collision sphere radius=0.005
