Commit message: changed 'package' to 'model'

File: pibot_description/models/iti0201_robot_cone/urdf/pibot_description.urdf.xacro (robot description, xacro)
@@ -16,5 +16,5 @@
         <origin xyz="0.0745 -0.0725 0.0025" rpy="0 0 1.57"/>
         <geometry>
-          <mesh filename="package://iti0201_robot/meshes/base_green.dae"/>
+          <mesh filename="model://iti0201_robot/meshes/base_green.dae"/>
           <!--cylinder length="0.0015" radius="0.07"/-->
         </geometry>
@@ -23,5 +23,5 @@
         <origin xyz="0.0745 -0.0725 0.0025" rpy="0 0 1.57"/>
         <geometry>
-          <mesh filename="package://iti0201_robot/meshes/base_green.dae"/>
+          <mesh filename="model://iti0201_robot/meshes/base_green.dae"/>
           <!--cylinder length="0.0015" radius="0.07"/-->
         </geometry>
