Commit message: should work

File: pibot_description/models/iti0201_robot/urdf/pibot_description.urdf.xacro (robot description, xacro)
@@ -1076,5 +1076,5 @@
 <!-- ARM -->
   <xacro:macro name="grabber_arm">
-    <link name="grabber_pole">
+    <link name="grabber_to_base_1">
       <inertial>
         <mass value="0.001"/>
@@ -1084,70 +1084,20 @@
       </inertial>
       <collision name="arm_to_base_col">
+        <geometry>
+          <box size=".006 .034 .03455"/>
+        </geometry>
+      </collision>
+      <visual name="arm_to_base_vis">
+        <geometry>
+          <box size=".006 .034 .03455"/>
+        </geometry>
+      </visual>
+    </link>
+    <joint type="fixed" name="grabber_to_base_joint_1">
       <origin xyz="0.055 0 0.0235" rpy="0 0 0" />
-        <geometry>
-          <box size=".006 .034 .03455"/>
-        </geometry>
-      </collision>
-      <visual name="arm_to_base_vis">
-      <origin xyz="0.055 0 0.0235" rpy="0 0 0" />
-        <geometry>
-          <box size=".006 .034 .03455"/>
-        </geometry>
-      </visual>
-      <collision name="collision_1">
-        <origin xyz="0.058912 0 0.0455477" rpy="0 1.5707 1.5707" />
-        <geometry>
-          <cylinder radius=".006" length=".034"/>
-        </geometry>
-      </collision>
-      <visual name="visual_1">
-        <origin xyz="0.058912 0 0.0455477" rpy="0 1.5707 1.5707" />
-        <geometry>
-          <cylinder radius=".006" length=".034"/>
-        </geometry>
-      </visual>
-    </link>
-    <joint type="fixed" name="grabber_pole">
-      <origin xyz="0 0 0" rpy="0 0 0" />
-      <child link="grabber_pole"/>
-      <parent link="base_with_casters"/>
-    </joint>
-    <link name="grabber_mount">
-      <collision name="arm_collision_left">
-        <origin xyz="0.073412 0.020 0.0455477" rpy="0 0 0" />
-        <geometry>
-          <box size=".035 .006 .011"/>
-        </geometry>
-      </collision>
-      <visual name="arm_visual_left">
-        <origin xyz="0.073412 0.020 0.0455477" rpy="0 0 0" />
-        <geometry>
-          <box size=".035 .006 .011"/>
-        </geometry>
-      </visual>
-      <collision name="arm_collision_right">
-        <origin xyz="0.073412 -0.020 0.0455477" rpy="0 0 0" />
-        <geometry>
-          <box size=".035 .006 .011"/>
-        </geometry>
-      </collision>
-      <visual name="arm_visual_right">
-        <origin xyz="0.073412 -0.020 0.0455477" rpy="0 0 0" />
-        <geometry>
-          <box size=".035 .006 .011"/>
-        </geometry>
-      </visual>
-      <collision name="collision_under">
-        <origin xyz="0.083912 0 0.0369977" rpy="0 0 0" />
-        <geometry>
-          <box size=".015 .042 .0057"/>
-        </geometry>
-      </collision>
-      <visual name="visual_under">
-        <origin xyz="0.083912 0 0.0369977" rpy="0 0 0" />
-        <geometry>
-          <box size=".015 .042 .0057"/>
-        </geometry>
-      </visual>
+      <child link="grabber_to_base_1"/>
+      <parent link="base_with_casters"/>
+    </joint>
+    <link name="pole_rotation_reference">
       <inertial>
         <mass value="0.001"/>
@@ -1156,28 +1106,21 @@
           izz="0.0000248"/>
       </inertial>
-    </link>
-      <!--
-      TODO: revolute?
-      -->
-    <joint type="revolute" name="grabber_mount_to_pole">
-      <origin xyz="0 0 0" rpy="0 0 0" />
-      <child link="grabber_mount"/>
-      <parent link="grabber_pole"/>
-      <limit effort="10.0" velocity="1.0" lower="0.0" upper="-1.5"/>
-      <axis xyz="0 1 0" />
-    </joint>
-    <link name="grabber_arms_joint">
-      <collision name="collision_for_arms_joint">
-      <origin xyz="0.083912 0 0.0319977" rpy="0 3.1414 0" />
-        <geometry>
-          <cylinder radius=".004" length=".005"/>
-        </geometry>
-      </collision>
-      <visual name="visual_for_arms_joint">
-      <origin xyz="0.083912 0 0.0319977" rpy="0 3.1414 0" />
-        <geometry>
-          <cylinder radius=".004" length=".005"/>
-        </geometry>
-      </visual>
+      <collision name="pole_rotation_reference_col">
+        <geometry>
+          <box size=".001 .001 .001"/>
+        </geometry>
+      </collision>
+      <visual name="pole_rotation_reference_vis">
+        <geometry>
+          <box size=".001 .001 .001"/>
+        </geometry>
+      </visual>
+    </link>
+    <joint type="fixed" name="pole_rotation_reference_to_base">
+      <origin xyz="0.059 0 0.04555" rpy="0 1.5707 1.5707" />
+      <child link="pole_rotation_reference"/>
+      <parent link="base_with_casters"/>
+    </joint>
+    <link name="grabber_pole">
       <inertial>
         <mass value="0.001"/>
@@ -1186,45 +1129,58 @@
           izz="0.0000248"/>
       </inertial>
-    </link>
-    <joint type="fixed" name="grabber_arms_joint_to_grabber_mount">
+      <collision name="the_pole_col">
+        <geometry>
+          <cylinder radius=".006" length=".034"/>
+        </geometry>
+      </collision>
+      <visual name="the_pole_vis">
+        <geometry>
+          <cylinder radius=".006" length=".034"/>
+        </geometry>
+      </visual>
+    </link>
+    <!-- TODO -->
+    <joint type="revolute" name="grabber_pole">
       <origin xyz="0 0 0" rpy="0 0 0" />
-      <child link="grabber_arms_joint"/>
-      <parent link="grabber_mount"/>
-    </joint>
-    <link name="grabber_arm_left">
-      <collision name="main_arm_collision_l">
-        <origin xyz="0.106912 0.022 0.0319977" rpy="0 0 0.78535"/>
-        <geometry>
-          <box size=".06213 .009 .005"/>
-        </geometry>
-      </collision>
-      <visual name="main_arm_visual_l">
-        <origin xyz="0.106912 0.022 0.0319977" rpy="0 0 0.78535"/>
-        <geometry>
-          <box size=".06213 .009 .005"/>
-        </geometry>
-      </visual>
-      <collision name="small_arm_collision_l_f">
-        <origin xyz="0.145 0.040 0.0294977" rpy="0 0 0"/>
-        <geometry>
-          <box size=".029 .003 .002"/>
-        </geometry>
-      </collision>
-      <visual name="small_arm_visual_l_f">
-        <origin xyz="0.145 0.040 0.0294977" rpy="0 0 0"/>
-        <geometry>
-          <box size=".029 .003 .002"/>
-        </geometry>
-      </visual>
-      <collision name="small_arm_collision_l_b">
-        <origin xyz="0.1305 0.0255 0.0294977" rpy="0 0 -1.5707"/>
-        <geometry>
-          <box size=".029 .003 .002"/>
-        </geometry>
-      </collision>
-      <visual name="small_arm_visual_l_b">
-        <origin xyz="0.1305 0.0255 0.0294977" rpy="0 0 -1.5707"/>
-        <geometry>
-          <box size=".029 .003 .002"/>
+      <child link="grabber_pole"/>
+      <parent link="pole_rotation_reference"/>
+      <limit effort="10.0" velocity="1.0" lower="0.0" upper="1.5"/>
+      <axis xyz="0 0 1"/>
+    </joint>
+    <link name="grabber_mount">
+      <collision name="arm_collision_left">
+        <origin xyz="0.0144 0.02 0" rpy="0 0 0" />
+        <geometry>
+          <box size=".035 .006 .011"/>
+        </geometry>
+      </collision>
+      <visual name="arm_visual_left">
+        <origin xyz="0.0144 0.02 0" rpy="0 0 0" />
+        <geometry>
+          <box size=".035 .006 .011"/>
+        </geometry>
+      </visual>
+      <collision name="arm_collision_right">
+        <origin xyz="0.0144 -0.02 0" rpy="0 0 0" />
+        <geometry>
+          <box size=".035 .006 .011"/>
+        </geometry>
+      </collision>
+      <visual name="arm_visual_right">
+        <origin xyz="0.0144 -0.02 0" rpy="0 0 0" />
+        <geometry>
+          <box size=".035 .006 .011"/>
+        </geometry>
+      </visual>
+      <collision name="collision_under">
+        <origin xyz="0.025 0 -0.00855" rpy="0 0 0"/>
+        <geometry>
+          <box size=".015 .042 .0057"/>
+        </geometry>
+      </collision>
+      <visual name="visual_under">
+        <origin xyz="0.025 0 -0.00855" rpy="0 0 0"/>
+        <geometry>
+          <box size=".015 .042 .0057"/>
         </geometry>
       </visual>
@@ -1236,49 +1192,18 @@
       </inertial>
     </link>
-      <!--
-      TODO: revolute?
-      -->
-    <joint type="revolute" name="grabber_arm_left_to_grabber_joint">
-      <origin xyz="0 0 0" rpy="0 0 0" />
-      <child link="grabber_arm_left"/>
-      <parent link="grabber_arms_joint"/>
-      <limit effort="10.0" velocity="1.0" lower="0.0" upper="0.8"/>
-      <axis xyz="0 0 1" />
-    </joint>
-    <link name="grabber_arm_right">
-      <collision name="main_arm_collision_r">
-        <origin xyz="0.106912 -0.022 0.0319977" rpy="0 0 -0.78535"/>
-        <geometry>
-          <box size=".06213 .009 .005"/>
-        </geometry>
-      </collision>
-      <visual name="main_arm_visual_r">
-        <origin xyz="0.106912 -0.022 0.0319977" rpy="0 0 -0.78535"/>
-        <geometry>
-          <box size=".06213 .009 .005"/>
-        </geometry>
-      </visual>
-      <collision name="small_arm_collision_r_f">
-        <origin xyz="0.145 -0.040 0.0294977" rpy="0 0 0"/>
-        <geometry>
-          <box size=".029 .003 .002"/>
-        </geometry>
-      </collision>
-      <visual name="small_arm_visual_r_f">
-        <origin xyz="0.145 -0.040 0.0294977" rpy="0 0 0"/>
-        <geometry>
-          <box size=".029 .003 .002"/>
-        </geometry>
-      </visual>
-      <collision name="small_arm_collision_r_b">
-        <origin xyz="0.1305 -0.0255 0.0294977" rpy="0 0 -1.5707"/>
-        <geometry>
-          <box size=".029 .003 .002"/>
-        </geometry>
-      </collision>
-      <visual name="small_arm_visual_r_b">
-        <origin xyz="0.1305 -0.0255 0.0294977" rpy="0 0 -1.5707"/>
-        <geometry>
-          <box size=".029 .003 .002"/>
+    <joint type="fixed" name="grabber_mount_to_pole">
+      <origin xyz="0 0 0" rpy="1.5707 0 3.1414"/>
+      <child link="grabber_mount"/>
+      <parent link="grabber_pole"/>
+    </joint>
+    <link name="grabber_left_arm_joint">
+      <collision name="collision_for_left_arm_joint">
+        <geometry>
+          <cylinder radius=".002" length=".004"/>
+        </geometry>
+      </collision>
+      <visual name="visual_for_left_arm_joint">
+        <geometry>
+          <cylinder radius=".002" length=".004"/>
         </geometry>
       </visual>
@@ -1290,13 +1215,135 @@
       </inertial>
     </link>
-      <!--
-      TODO: revolute?
-      -->
-    <joint type="revolute" name="grabber_arm_right_to_grabber_joint">
-      <limit effort="10.0" velocity="1.0" lower="0.0" upper="0.8" />
-      <origin xyz="0 0 0" rpy="0 0 0" />
+    <!-- TODO -->
+    <joint type="revolute" name="grabber_left_arm_joint_to_grabber_mount">
+      <origin xyz="0.025 0.01 -0.01355" rpy="0 3.1414 0" />
+      <child link="grabber_left_arm_joint"/>
+      <parent link="grabber_mount"/>
+      <limit effort="10.0" velocity="1.0" lower="0.0" upper="0.7"/>
+      <axis xyz="0 0 1"/>
+    </joint>
+    <link name="grabber_right_arm_joint">
+      <collision name="collision_for_right_arm_joint">
+        <geometry>
+          <cylinder radius=".002" length=".004"/>
+        </geometry>
+      </collision>
+      <visual name="visual_for_right_arm_joint">
+        <geometry>
+          <cylinder radius=".002" length=".004"/>
+        </geometry>
+      </visual>
+      <inertial>
+        <mass value="0.001"/>
+        <inertia ixx="0.0000337" ixy="0.0" ixz="0.0"
+          iyy="0.0000493" iyz="0.0"
+          izz="0.0000248"/>
+      </inertial>
+    </link>
+    <!-- TODO -->
+    <joint type="revolute" name="grabber_right_arm_joint_to_grabber_mount">
+      <origin xyz="0.025 -0.01 -0.01355" rpy="0 3.1414 0" />
+      <child link="grabber_right_arm_joint"/>
+      <parent link="grabber_mount"/>
+      <limit effort="10.0" velocity="1.0" lower="0.0" upper="-0.7"/>
+      <axis xyz="0 0 1"/>
+    </joint>
+    <link name="grabber_arm_left">
+      <collision name="main_arm_collision_l">
+        <origin xyz="0.023 0.019 0" rpy="0 0 0.78535"/>
+        <geometry>
+          <box size=".06213 .009 .005"/>
+        </geometry>
+      </collision>
+      <visual name="main_arm_visual_l">
+        <origin xyz="0.023 0.019 0" rpy="0 0 0.78535"/>
+        <geometry>
+          <box size=".06213 .009 .005"/>
+        </geometry>
+      </visual>
+      <collision name="small_arm_collision_l_f">
+        <origin xyz="0.061 0.037 -0.0025" rpy="0 0 0"/>
+        <geometry>
+          <box size=".029 .003 .002"/>
+        </geometry>
+      </collision>
+      <visual name="small_arm_visual_l_f">
+        <origin xyz="0.061 0.037 -0.0025" rpy="0 0 0"/>
+        <geometry>
+          <box size=".029 .003 .002"/>
+        </geometry>
+      </visual>
+      <collision name="small_arm_collision_l_b">
+        <origin xyz="0.0465 0.0225 -0.0025" rpy="0 0 -1.5707"/>
+        <geometry>
+          <box size=".029 .003 .002"/>
+        </geometry>
+      </collision>
+      <visual name="small_arm_visual_l_b">
+        <origin xyz="0.0465 0.0225 -0.0025" rpy="0 0 -1.5707"/>
+        <geometry>
+          <box size=".029 .003 .002"/>
+        </geometry>
+      </visual>
+      <inertial>
+        <mass value="0.001"/>
+        <inertia ixx="0.0000337" ixy="0.0" ixz="0.0"
+          iyy="0.0000493" iyz="0.0"
+          izz="0.0000248"/>
+      </inertial>
+    </link>
+    <joint type="fixed" name="grabber_arm_left_to_grabber_joint">
+      <origin xyz="0 0 0" rpy="0 3.1414 0" />
+      <child link="grabber_arm_left"/>
+      <parent link="grabber_left_arm_joint"/>
+    </joint>
+    <link name="grabber_arm_right">
+      <collision name="main_arm_collision_r">
+        <origin xyz="0.023 -0.019 0" rpy="0 0 -0.78535"/>
+        <geometry>
+          <box size=".06213 .009 .005"/>
+        </geometry>
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
Commit message: update xacro

File: pibot_description/models/iti0201_robot/urdf/pibot_description.urdf.xacro (robot description, xacro)
@@ -14,5 +14,5 @@
       </inertial>
       <visual name="base_visual">
-        <origin xyz="-0.09 0.098 0.005" rpy="0 0 -1.57"/>
+        <origin xyz="-0.0615 0.098 0.005" rpy="0 0 -1.57"/>
         <geometry>
           <mesh filename="model://iti0201_robot/meshes/pibot2_base.dae"/>
@@ -21,5 +21,5 @@
       </visual>
       <collision name="base_collision">
-        <origin xyz="-0.09 0.098 0.005" rpy="0 0 -1.57"/>
+        <origin xyz="-0.0615 0.098 0.005" rpy="0 0 -1.57"/>
         <geometry>
           <mesh filename="model://iti0201_robot/meshes/pibot2_base.dae"/>
@@ -66,5 +66,5 @@
     </link>
     <joint type="fixed" name="Wheel_joint_to_base">
-      <origin xyz="-0.0285 0 0.015" rpy="0 0 0" />
+      <origin xyz="0 0 0.015" rpy="0 0 0" />
       <child link="wheel_joint"/>
       <parent link="base_with_casters" />
@@ -106,5 +106,5 @@
     </link>
     <joint type="fixed" name="brainbox_to_base">
-      <origin xyz="0 0 0.003" rpy="0 0 0"/>
+      <origin xyz="0.0285 0 0.003" rpy="0 0 0"/>
       <child link="brainbox_with_battery"/>
       <parent link="base_with_casters"/>
@@ -132,5 +132,5 @@
     </link>
     <joint type="fixed" name="front_right_45deg_ir_to_base">
-      <origin xyz="0.0326 -0.0471 0.016" rpy="0 0 -0.78535"/>
+      <origin xyz="0.0611 -0.0471 0.016" rpy="0 0 -0.78535"/>
       <child link="front_right_45deg_ir"/>
       <parent link="base_with_casters"/>
@@ -178,5 +178,5 @@
     </link>
     <joint type="fixed" name="front_middle_ir_to_base">
-      <origin xyz="0.059312 0 0.011" rpy="0 0 0"/>
+      <origin xyz="0.087812 0 0.011" rpy="0 0 0"/>
       <child link="front_middle_ir"/>
       <parent link="base_with_casters"/>
@@ -224,5 +224,5 @@
     </link>
     <joint type="fixed" name="front_left_45deg_ir_to_base">
-      <origin xyz="0.0326151 0.0470558 0.016" rpy="0 0 0.78535"/>
+      <origin xyz="0.0611151 0.0470558 0.016" rpy="0 0 0.78535"/>
       <child link="front_left_45deg_ir"/>
       <parent link="base_with_casters"/>
@@ -273,5 +273,5 @@
     </link>
     <joint type="fixed" name="rear_right_90deg_ir_to_base">
-      <origin xyz="-0.05 -0.058 0.013" rpy="0 0 -1.5707" />
+      <origin xyz="-0.0215 -0.058 0.013" rpy="0 0 -1.5707" />
       <child link="rear_right_90deg_ir"/>
       <parent link="base_with_casters"/>
@@ -319,5 +319,5 @@
     </link>
     <joint type="fixed" name="rear_right_45deg_ir_to_base">
-      <origin xyz="-0.0585 -0.045 0.013" rpy="0 0 -2.35605" />
+      <origin xyz="-0.03 -0.045 0.013" rpy="0 0 -2.35605" />
       <child link="rear_right_45deg_ir"/>
       <parent link="base_with_casters"/>
@@ -365,5 +365,5 @@
     </link>
     <joint type="fixed" name="rear_right_straight_ir_to_base">
-      <origin xyz="-0.06 -0.03 0.013" rpy="0 0 -3.14" />
+      <origin xyz="-0.0315 -0.03 0.013" rpy="0 0 -3.14" />
       <child link="rear_right_straight_ir"/>
       <parent link="base_with_casters"/>
@@ -411,5 +411,5 @@
     </link>
     <joint type="fixed" name="rear_left_90deg_ir_to_base">
-      <origin xyz="-0.05 0.058 0.013" rpy="0 0 1.5707" />
+      <origin xyz="-0.0215 0.058 0.013" rpy="0 0 1.5707" />
       <child link="rear_left_90deg_ir"/>
       <parent link="base_with_casters"/>
@@ -457,5 +457,5 @@
     </link>
     <joint type="fixed" name="rear_left_45deg_ir_to_base">
-      <origin xyz="-0.0585 0.045 0.013" rpy="0 0 2.35605" />
+      <origin xyz="-0.03 0.045 0.013" rpy="0 0 2.35605" />
       <child link="rear_left_45deg_ir"/>
       <parent link="base_with_casters"/>
@@ -503,5 +503,5 @@
     </link>
     <joint type="fixed" name="rear_left_straight_ir_to_base">
-      <origin xyz="-0.06 0.03 0.013" rpy="0 0 3.14" />
+      <origin xyz="-0.0315 0.03 0.013" rpy="0 0 3.14" />
       <child link="rear_left_straight_ir"/>
       <parent link="base_with_casters"/>
@@ -553,5 +553,5 @@
     </link>
     <joint type="fixed" name="right_side_first_line_sensor_from_middle_to_base">
-      <origin xyz="0.065 -0.005 0.0044" rpy="0 1.5707 0" />
+      <origin xyz="0.0935 -0.005 0.0044" rpy="0 1.5707 0" />
       <child link="right_side_first_line_sensor_from_middle"/>
       <parent link="base_with_casters"/>
@@ -610,5 +610,5 @@
     </link>
     <joint type="fixed" name="left_side_first_line_sensor_from_middle_to_base">
-      <origin xyz="0.065 0.005 0.0044" rpy="0 1.5707 0" />
+      <origin xyz="0.0935 0.005 0.0044" rpy="0 1.5707 0" />
       <child link="left_side_first_line_sensor_from_middle"/>
       <parent link="base_with_casters"/>
@@ -670,5 +670,5 @@
     </link>
     <joint type="fixed" name="right_side_second_line_sensor_from_middle_to_base">
-      <origin xyz="0.065 -0.015 0.0044" rpy="0 1.5707 0" />
+      <origin xyz="0.0935 -0.015 0.0044" rpy="0 1.5707 0" />
       <child link="right_side_second_line_sensor_from_middle"/>
       <parent link="base_with_casters"/>
@@ -728,5 +728,5 @@
     </link>
     <joint type="fixed" name="left_side_second_line_sensor_from_middle_to_base">
-      <origin xyz="0.065 0.015 0.0044" rpy="0 1.5707 0" />
+      <origin xyz="0.0935 0.015 0.0044" rpy="0 1.5707 0" />
       <child link="left_side_second_line_sensor_from_middle"/>
       <parent link="base_with_casters"/>
@@ -788,5 +788,5 @@
     </link>
     <joint type="fixed" name="right_side_third_line_sensor_from_middle_to_base">
-      <origin xyz="0.057 -0.035 0.0044" rpy="0 1.5707 0" />
+      <origin xyz="0.0855 -0.035 0.0044" rpy="0 1.5707 0" />
       <child link="right_side_third_line_sensor_from_middle"/>
       <parent link="base_with_casters"/>
@@ -846,5 +846,5 @@
     </link>
     <joint type="fixed" name="left_side_third_line_sensor_from_middle_to_base">
-      <origin xyz="0.057 0.035 0.0044" rpy="0 1.5707 0" />
+      <origin xyz="0.0855 0.035 0.0044" rpy="0 1.5707 0" />
       <child link="left_side_third_line_sensor_from_middle"/>
       <parent link="base_with_casters"/>
@@ -907,5 +907,5 @@
     </link>
     <joint type="fixed" name="camera_stand_pole_to_base">
-      <origin xyz="0.02940475 0 0.1135341" rpy="0 1.5707 1.5707" />
+      <origin xyz="0.05790475 0 0.1135341" rpy="0 1.5707 1.5707" />
       <child link="camera_stand_pole"/>
       <parent link="base_with_casters"/>
@@ -1077,5 +1077,5 @@
     </link>
     <joint type="fixed" name="grabber_to_base_joint_1">
-      <origin xyz="0.055 0 0.0235" rpy="0 0 0" />
+      <origin xyz="0.0835 0 0.0235" rpy="0 0 0" />
       <child link="grabber_to_base_1"/>
       <parent link="base_with_casters"/>
@@ -1100,5 +1100,5 @@
     </link>
     <joint type="fixed" name="pole_rotation_reference_to_base">
-      <origin xyz="0.059 0 0.04555" rpy="0 1.5707 1.5707" />
+      <origin xyz="0.0875 0 0.04555" rpy="0 1.5707 1.5707" />
       <child link="pole_rotation_reference"/>
       <parent link="base_with_casters"/>
