Commit message: Grabber stuff

File: pibot_description/models/iti0201_robot/urdf/pibot.urdf (robot description, URDF)
Before this commit: robot pibot, 27 links, 26 joints
Joints:
- joint grabber_arm_left_to_grabber_joint: axis (none) -> 0 0 1; limit (none) -> lower=0.0 upper=0.8 effort=10.0 velocity=1.0; type fixed -> revolute
- joint grabber_arm_right_to_grabber_joint: axis (none) -> 0 0 1; limit (none) -> lower=0.0 upper=0.8 effort=10.0 velocity=1.0; type fixed -> revolute
- joint grabber_mount_to_pole: axis (none) -> 0 1 0; limit (none) -> lower=0.0 upper=-1.5 effort=10.0 velocity=1.0; type fixed -> revolute

File: pibot_description/models/iti0201_robot/urdf/pibot_description.urdf.xacro (robot description, xacro)
@@ -1160,8 +1160,10 @@
       TODO: revolute?
       -->
-    <joint type="fixed" name="grabber_mount_to_pole">
+    <joint type="revolute" name="grabber_mount_to_pole">
       <origin xyz="0 0 0" rpy="0 0 0" />
       <child link="grabber_mount"/>
       <parent link="grabber_pole"/>
+      <limit effort="10.0" velocity="1.0" lower="0.0" upper="-1.5"/>
+      <axis xyz="0 1 0" />
     </joint>
     <link name="grabber_arms_joint">
@@ -1237,8 +1239,10 @@
       TODO: revolute?
       -->
-    <joint type="fixed" name="grabber_arm_left_to_grabber_joint">
+    <joint type="revolute" name="grabber_arm_left_to_grabber_joint">
       <origin xyz="0 0 0" rpy="0 0 0" />
       <child link="grabber_arm_left"/>
       <parent link="grabber_arms_joint"/>
+      <limit effort="10.0" velocity="1.0" lower="0.0" upper="0.8"/>
+      <axis xyz="0 0 1" />
     </joint>
     <link name="grabber_arm_right">
@@ -1289,9 +1293,14 @@
       TODO: revolute?
       -->
-    <joint type="fixed" name="grabber_arm_right_to_grabber_joint">
+    <joint type="revolute" name="grabber_arm_right_to_grabber_joint">
+      <limit effort="10.0" velocity="1.0" lower="0.0" upper="0.8" />
       <origin xyz="0 0 0" rpy="0 0 0" />
       <child link="grabber_arm_right"/>
       <parent link="grabber_arms_joint"/>
-    </joint>
+      <axis xyz="0 0 1" />
+    </joint>
+    <gazebo>
+      <plugin name="grabber_plugin" filename="libgrabber_plugin.so"/>
+    </gazebo>
   </xacro:macro>
 </robot>

Commit message: Fixed grabber plugin

File: pibot_description/models/iti0201_robot/urdf/pibot.urdf (robot description, URDF)
Before this commit: robot pibot, 27 links, 26 joints
Links:
- added link brainbox_with_battery, mass 0.001; visual box size=0.0255 0.006 0.0346; visual box size=0.0255 0.006 0.0346
- added link camera_stand_pole, mass 0.001; collision cylinder length=0.0433499 radius=0.003822; visual cylinder length=0.0433499 radius=0.003822
- added link pi_camera, mass 0.001; collision box size=0.017 0.024 0.024; visual box size=0.017 0.024 0.024
Joints:
- added joint brainbox_to_base: type fixed, parent base_with_casters, child brainbox_with_battery, origin xyz=0 0 0 rpy=0 0 0
- added joint camera_stand_pole_to_base: type fixed, parent base_with_casters, child camera_stand_pole, origin xyz=0.02940475 0 0.1135341 rpy=0 1.5707 1.5707
- added joint pi_camera_to_pole: type fixed, parent camera_stand_pole, child pi_camera, origin xyz=0 -0.0104 0 rpy=0 0 -1.5707

Commit message: fdir + kp + incr mu

File: pibot_description/models/iti0201_robot/urdf/pibot.urdf (robot description, URDF)
Before this commit: robot pibot, 28 links, 27 joints
Links:
- added link camera_stand_pole, mass 0.001; collision cylinder length=0.0433499 radius=0.003822; visual cylinder length=0.0433499 radius=0.003822
- added link pi_camera, mass 0.001; collision box size=0.017 0.024 0.024; visual box size=0.017 0.024 0.024
Joints:
- added joint camera_stand_pole_to_base: type fixed, parent base_with_casters, child camera_stand_pole, origin xyz=0.02940475 0 0.1135341 rpy=0 1.5707 1.5707
- added joint pi_camera_to_pole: type fixed, parent camera_stand_pole, child pi_camera, origin xyz=0 -0.0104 0 rpy=0 0 -1.5707

File: pibot_description/models/iti0201_robot/urdf/pibot_description.urdf.xacro (robot description, xacro)
@@ -1012,14 +1012,9 @@
     </link>
     <gazebo reference="right_wheel">
-      <surface>
-          <friction>
-             <ode>
-                <!-- wheel friction coefficient -->
-                <mu>0.6</mu>
-                <!-- floor friction coefficient -->
-                <mu2>0.6</mu2>
-             </ode>
-          </friction>
-        </surface>
+      <mu1 value="1.0"/>
+      <mu2 value="1.0"/>
+      <kp value="10000000.0" />
+      <kd value="1.0" />
+      <fdir1 value="1 0 0"/>
     </gazebo>
     <joint type="continuous" name="right_wheel_hinge">
@@ -1052,14 +1047,9 @@
     </link>
     <gazebo reference="left_wheel">
-      <surface>
-          <friction>
-             <ode>
-                <!-- wheel friction coefficient -->
-                <mu>0.6</mu>
-                <!-- floor friction coefficient -->
-                <mu2>0.6</mu2>
-             </ode>
-          </friction>
-        </surface>
+      <mu1 value="1.0"/>
+      <mu2 value="1.0"/>
+      <kp value="10000000.0" />
+      <kd value="1.0" />
+      <fdir1 value="1 0 0"/>
     </gazebo>
     <joint type="continuous" name="left_wheel_hinge">

Commit message: robot fix

File: pibot_description/models/iti0201_robot/urdf/pibot.urdf (robot description, URDF)
Before this commit: robot pibot, 30 links, 29 joints
Links:
- link base_with_casters: mass 0.48 -> 5
- link left_wheel: mass 0.005 -> 1
- link right_wheel: mass 0.005 -> 1

File: pibot_description/models/iti0201_robot/urdf/pibot_description.urdf.xacro (robot description, xacro)
@@ -4,5 +4,5 @@
     <xacro:property name="base_radius" value="0.07" />
     <xacro:property name="base_height" value="0.0015" />
-    <xacro:property name="base_mass" value="0.48" />
+    <xacro:property name="base_mass" value="5" /> <!--real: 0.48kg-->
     <xacro:property name="caster_wheel_radius" value="0.005" />
     <link name="base_with_casters">
@@ -990,5 +990,5 @@
 <!-- WHEELS -->
   <xacro:macro name="wheels">
-    <xacro:property name="wheel_mass" value="0.005" />
+    <xacro:property name="wheel_mass" value="1" /> <!-- real: 0.005-->
     <xacro:property name="wheel_radius" value="0.0125"/>
     <xacro:property name="wheel_length" value="0.009"/>

Commit message: Changed reference from 'package' to 'model'

File: pibot_description/models/iti0201_robot/urdf/pibot.urdf (robot description, URDF)
Before this commit: robot pibot, 28 links, 27 joints
Links:
- link base_with_casters: geometry collision mesh filename=model://iti0201_robot/meshes/base_green.dae; collision sphere radius=0.005

File: pibot_description/models/iti0201_robot/urdf/pibot_description.urdf.xacro (robot description, xacro)
@@ -16,5 +16,5 @@
         <origin xyz="0.0745 -0.0725 0.0025" rpy="0 0 1.57"/>
         <geometry>
-          <mesh filename="package://iti0201_robot/meshes/base_green.dae"/>
+          <mesh filename="model://iti0201_robot/meshes/base_green.dae"/>
           <!--cylinder length="0.0015" radius="0.07"/-->
         </geometry>
@@ -23,5 +23,5 @@
         <origin xyz="0.0745 -0.0725 0.0025" rpy="0 0 1.57"/>
         <geometry>
-          <mesh filename="package://iti0201_robot/meshes/base_green.dae"/>
+          <mesh filename="model://iti0201_robot/meshes/base_green.dae"/>
           <!--cylinder length="0.0015" radius="0.07"/-->
         </geometry>

Commit message: Update pibot.urdf

File: pibot_description/models/iti0201_robot/urdf/pibot.urdf (robot description, URDF)
Before this commit: robot pibot, 28 links, 27 joints
Links:
- link base_with_casters: geometry collision mesh filename=package://iti0201_robot/meshes/base_green.dae; collision sphere radius=0.005

Commit message: Line sensors to front

File: pibot_description/models/iti0201_robot/urdf/pibot.urdf (robot description, URDF)
Before this commit: robot pibot, 30 links, 29 joints
Joints:
- joint left_side_first_line_sensor_from_middle_to_base: origin xyz=-0.0629 0.005 0.0044 rpy=0 1.5707 0 -> xyz=0.065 0.005 0.0044 rpy=0 1.5707 0
- joint left_side_second_line_sensor_from_middle_to_base: origin xyz=-0.06289935 0.015 0.0044 rpy=0 1.5707 0 -> xyz=0.065 0.015 0.0044 rpy=0 1.5707 0
- joint left_side_third_line_sensor_from_middle_to_base: origin xyz=-0.0541 0.035 0.0044 rpy=0 1.5707 0 -> xyz=0.057 0.035 0.0044 rpy=0 1.5707 0
- joint right_side_first_line_sensor_from_middle_to_base: origin xyz=-0.0629 -0.005 0.0044 rpy=0 1.5707 0 -> xyz=0.065 -0.005 0.0044 rpy=0 1.5707 0
- joint right_side_second_line_sensor_from_middle_to_base: origin xyz=-0.06289935 -0.015 0.0044 rpy=0 1.5707 0 -> xyz=0.065 -0.015 0.0044 rpy=0 1.5707 0
- joint right_side_third_line_sensor_from_middle_to_base: origin xyz=-0.0541 -0.035 0.0044 rpy=0 1.5707 0 -> xyz=0.057 -0.035 0.0044 rpy=0 1.5707 0

File: pibot_description/models/iti0201_robot/urdf/pibot_description.urdf.xacro (robot description, xacro)
@@ -553,5 +553,5 @@
     </link>
     <joint type="fixed" name="right_side_first_line_sensor_from_middle_to_base">
-      <origin xyz="-0.0629 -0.005 0.0044" rpy="0 1.5707 0" />
+      <origin xyz="0.065 -0.005 0.0044" rpy="0 1.5707 0" />
       <child link="right_side_first_line_sensor_from_middle"/>
       <parent link="base_with_casters"/>
@@ -610,5 +610,5 @@
     </link>
     <joint type="fixed" name="left_side_first_line_sensor_from_middle_to_base">
-      <origin xyz="-0.0629 0.005 0.0044" rpy="0 1.5707 0" />
+      <origin xyz="0.065 0.005 0.0044" rpy="0 1.5707 0" />
       <child link="left_side_first_line_sensor_from_middle"/>
       <parent link="base_with_casters"/>
@@ -670,5 +670,5 @@
     </link>
     <joint type="fixed" name="right_side_second_line_sensor_from_middle_to_base">
-      <origin xyz="-0.06289935 -0.015 0.0044" rpy="0 1.5707 0" />
+      <origin xyz="0.065 -0.015 0.0044" rpy="0 1.5707 0" />
       <child link="right_side_second_line_sensor_from_middle"/>
       <parent link="base_with_casters"/>
@@ -728,5 +728,5 @@
     </link>
     <joint type="fixed" name="left_side_second_line_sensor_from_middle_to_base">
-      <origin xyz="-0.06289935 0.015 0.0044" rpy="0 1.5707 0" />
+      <origin xyz="0.065 0.015 0.0044" rpy="0 1.5707 0" />
       <child link="left_side_second_line_sensor_from_middle"/>
       <parent link="base_with_casters"/>
@@ -788,5 +788,5 @@
     </link>
     <joint type="fixed" name="right_side_third_line_sensor_from_middle_to_base">
-      <origin xyz="-0.0541 -0.035 0.0044" rpy="0 1.5707 0" />
+      <origin xyz="0.057 -0.035 0.0044" rpy="0 1.5707 0" />
       <child link="right_side_third_line_sensor_from_middle"/>
       <parent link="base_with_casters"/>
@@ -846,5 +846,5 @@
     </link>
     <joint type="fixed" name="left_side_third_line_sensor_from_middle_to_base">
-      <origin xyz="-0.0541 0.035 0.0044" rpy="0 1.5707 0" />
+      <origin xyz="0.057 0.035 0.0044" rpy="0 1.5707 0" />
       <child link="left_side_third_line_sensor_from_middle"/>
       <parent link="base_with_casters"/>

Commit message: Hotfix Gazebo bugged physics

File: pibot_description/models/iti0201_robot/urdf/pibot.urdf (robot description, URDF)
Before this commit: robot pibot, 30 links, 29 joints
Joints:
- joint Wheel_joint_to_base: origin xyz=-0.0285 0 0.015 rpy=0 0 0 -> xyz=0 0 0.015 rpy=0 0 0
- joint brainbox_to_base: origin xyz=0 0 0.003 rpy=0 0 0 -> xyz=0.0285 0 0.003 rpy=0 0 0
- joint camera_stand_pole_to_base: origin xyz=0.02940475 0 0.1135341 rpy=0 1.5707 1.5707 -> xyz=0.05790475 0 0.1135341 rpy=0 1.5707 1.5707
- joint front_left_45deg_ir_to_base: origin xyz=0.0326151 0.0470558 0.016 rpy=0 0 0.78535 -> xyz=0.0611151 0.0470558 0.016 rpy=0 0 0.78535
- joint front_middle_ir_to_base: origin xyz=0.059312 0 0.011 rpy=0 0 0 -> xyz=0.087812 0 0.011 rpy=0 0 0
- joint front_right_45deg_ir_to_base: origin xyz=0.0326 -0.0471 0.016 rpy=0 0 -0.78535 -> xyz=0.0611 -0.0471 0.016 rpy=0 0 -0.78535
- joint grabber_to_base_joint_1: origin xyz=0.055 0 0.0235 rpy=0 0 0 -> xyz=0.0835 0 0.0235 rpy=0 0 0
- joint left_side_first_line_sensor_from_middle_to_base: origin xyz=0.065 0.005 0.0044 rpy=0 1.5707 0 -> xyz=0.0935 0.005 0.0044 rpy=0 1.5707 0
- joint left_side_second_line_sensor_from_middle_to_base: origin xyz=0.065 0.015 0.0044 rpy=0 1.5707 0 -> xyz=0.0935 0.015 0.0044 rpy=0 1.5707 0
- joint left_side_third_line_sensor_from_middle_to_base: origin xyz=0.057 0.035 0.0044 rpy=0 1.5707 0 -> xyz=0.0855 0.035 0.0044 rpy=0 1.5707 0
- joint pole_rotation_reference_to_base: origin xyz=0.059 0 0.04555 rpy=0 1.5707 1.5707 -> xyz=0.0875 0 0.04555 rpy=0 1.5707 1.5707
- joint rear_left_45deg_ir_to_base: origin xyz=-0.0585 0.045 0.013 rpy=0 0 2.35605 -> xyz=-0.03 0.045 0.013 rpy=0 0 2.35605
- joint rear_left_90deg_ir_to_base: origin xyz=-0.05 0.058 0.013 rpy=0 0 1.5707 -> xyz=-0.0215 0.058 0.013 rpy=0 0 1.5707
- joint rear_left_straight_ir_to_base: origin xyz=-0.06 0.03 0.013 rpy=0 0 3.14 -> xyz=-0.0315 0.03 0.013 rpy=0 0 3.14
- joint rear_right_45deg_ir_to_base: origin xyz=-0.0585 -0.045 0.013 rpy=0 0 -2.35605 -> xyz=-0.03 -0.045 0.013 rpy=0 0 -2.35605
- joint rear_right_90deg_ir_to_base: origin xyz=-0.05 -0.058 0.013 rpy=0 0 -1.5707 -> xyz=-0.0215 -0.058 0.013 rpy=0 0 -1.5707
- joint rear_right_straight_ir_to_base: origin xyz=-0.06 -0.03 0.013 rpy=0 0 -3.14 -> xyz=-0.0315 -0.03 0.013 rpy=0 0 -3.14
- joint right_side_first_line_sensor_from_middle_to_base: origin xyz=0.065 -0.005 0.0044 rpy=0 1.5707 0 -> xyz=0.0935 -0.005 0.0044 rpy=0 1.5707 0
- joint right_side_second_line_sensor_from_middle_to_base: origin xyz=0.065 -0.015 0.0044 rpy=0 1.5707 0 -> xyz=0.0935 -0.015 0.0044 rpy=0 1.5707 0
- joint right_side_third_line_sensor_from_middle_to_base: origin xyz=0.057 -0.035 0.0044 rpy=0 1.5707 0 -> xyz=0.0855 -0.035 0.0044 rpy=0 1.5707 0

Commit message: Camera changes

File: pibot_description/models/iti0201_robot/urdf/pibot.urdf (robot description, URDF)
Before this commit: robot pibot, 30 links, 29 joints
Joints:
- joint pi_camera_to_pole: origin xyz=0 -0.0104 0 rpy=0 0 -1.5707 -> xyz=0 -0.0104 0 rpy=0 0 -1.1707

File: pibot_description/models/iti0201_robot/urdf/pibot_description.urdf.xacro (robot description, xacro)
@@ -940,5 +940,5 @@
     </link>
     <joint type="fixed" name="pi_camera_to_pole">
-      <origin xyz="0 -0.0104 0" rpy="0 0 -1.5707"/>
+      <origin xyz="0 -0.0104 0" rpy="0 0 -1.1707"/>
       <child link="pi_camera"/>
       <parent link="camera_stand_pole"/>
@@ -950,8 +950,8 @@
         <visualize>false</visualize>
         <camera name="head">
-          <horizontal_fov>1.3962634</horizontal_fov>
+          <horizontal_fov>1.09</horizontal_fov>
           <image>
-            <width>800</width>
-            <height>800</height>
+            <width>1080</width>
+            <height>1080</height>
             <format>R8G8B8</format>
           </image>

Commit message: Find single blue and red sphere with OpenCV

File: pibot_description/models/iti0201_robot/urdf/pibot.urdf (robot description, URDF)
Before this commit: robot pibot, 30 links, 29 joints
Joints:
- joint pi_camera_to_pole: origin xyz=0 -0.0104 0 rpy=0 0 -1.1707 -> xyz=0. -0.0104 0 rpy=1.5708 0 -1.1707

File: pibot_description/models/iti0201_robot/urdf/pibot_description.urdf.xacro (robot description, xacro)
@@ -940,5 +940,5 @@
     </link>
     <joint type="fixed" name="pi_camera_to_pole">
-      <origin xyz="0 -0.0104 0" rpy="0 0 -1.1707"/>
+      <origin xyz="0. -0.0104 0" rpy="1.5708 0 -1.1707"/>
       <child link="pi_camera"/>
       <parent link="camera_stand_pole"/>
@@ -954,5 +954,5 @@
             <width>1080</width>
             <height>1080</height>
-            <format>R8G8B8</format>
+            <format>B8G8R8</format>
           </image>
           <clip>

Commit message: Fix link name collision

File: pibot_description/models/iti0201_robot/urdf/pibot.urdf (robot description, URDF)
Before this commit: robot pibot, 30 links, 29 joints
Links:
- removed link grabber_pole
- added link grabber_pole_link, mass 0.001; collision cylinder length=.034 radius=.006; visual cylinder length=.034 radius=.006
Joints:
- joint grabber_mount_to_pole: parent grabber_pole -> grabber_pole_link
- joint grabber_pole: child grabber_pole -> grabber_pole_link

File: pibot_description/models/iti0201_robot/urdf/pibot_description.urdf.xacro (robot description, xacro)
@@ -1104,5 +1104,5 @@
       <parent link="base_with_casters"/>
     </joint>
-    <link name="grabber_pole">
+    <link name="grabber_pole_link">
       <inertial>
         <mass value="0.001"/>
@@ -1125,5 +1125,5 @@
     <joint type="revolute" name="grabber_pole">
       <origin xyz="0 0 0" rpy="0 0 0" />
-      <child link="grabber_pole"/>
+      <child link="grabber_pole_link"/>
       <parent link="pole_rotation_reference"/>
       <limit effort="10.0" velocity="1.0" lower="0.0" upper="1.5"/>
@@ -1177,5 +1177,5 @@
       <origin xyz="0 0 0" rpy="1.5707 0 3.1414"/>
       <child link="grabber_mount"/>
-      <parent link="grabber_pole"/>
+      <parent link="grabber_pole_link"/>
     </joint>
     <link name="grabber_left_arm_joint">
