Commit message: Changed robot base, removed raspberry camera from urdf to boost simulation performance

File: pibot_description/models/iti0201_robot/urdf/generate_pibot.urdf.xacro (robot description, xacro)
@@ -9,5 +9,5 @@
   <xacro:second_two_line_sensors/>
   <xacro:third_two_line_sensors/>
-  <xacro:raspberry_camera/>
+  <!--xacro:raspberry_camera/-->
   <xacro:wheels/>
   <xacro:grabber_arm/>

File: pibot_description/models/iti0201_robot/urdf/pibot.urdf (robot description, URDF)
Before this commit: robot pibot, 30 links, 29 joints
Links:
- removed link camera_stand_pole
- removed link pi_camera
- link base_with_casters: geometry collision mesh filename=package://iti0201_robot/meshes/base_green.dae; collision sphere radius=0.005
Joints:
- removed joint camera_stand_pole_to_base
- removed joint pi_camera_to_pole

File: pibot_description/models/iti0201_robot/urdf/pibot_description.urdf.xacro (robot description, xacro)
@@ -13,14 +13,16 @@
           izz="${1/2 * base_mass * (base_radius * base_radius)}"/>
       </inertial>
-      <visual name='base_visual'>
-      <origin xyz="0 0 0.003" rpy="0 0 0"/>
-        <geometry>
-          <cylinder radius="${base_radius}" length="${base_height}"/>
-        </geometry>
-      </visual>
-      <collision name='base_collision'>
-      <origin xyz="0 0 0.003" rpy="0 0 0"/>
-        <geometry>
-          <cylinder radius="${base_radius}" length="${base_height}"/>
+      <visual name="base_visual">
+        <origin xyz="0.0745 -0.0725 0.0025" rpy="0 0 1.57"/>
+        <geometry>
+          <mesh filename="package://iti0201_robot/meshes/base_green.dae"/>
+          <!--cylinder length="0.0015" radius="0.07"/-->
+        </geometry>
+      </visual>
+      <collision name="base_collision">
+        <origin xyz="0.0745 -0.0725 0.0025" rpy="0 0 1.57"/>
+        <geometry>
+          <mesh filename="package://iti0201_robot/meshes/base_green.dae"/>
+          <!--cylinder length="0.0015" radius="0.07"/-->
         </geometry>
       </collision>

File: pibot_description/models/iti0201_robot_cone/urdf/generate_pibot.urdf.xacro (robot description, xacro)
@@ -9,5 +9,5 @@
   <xacro:second_two_line_sensors/>
   <xacro:third_two_line_sensors/>
-  <xacro:raspberry_camera/>
+  <!--xacro:raspberry_camera/-->
   <xacro:wheels/>
   <xacro:grabber_arm/>

File: pibot_description/models/iti0201_robot_cone/urdf/pibot.urdf (robot description, URDF)
Before this commit: robot pibot, 30 links, 29 joints
Links:
- removed link camera_stand_pole
- removed link pi_camera
- link base_with_casters: geometry collision mesh filename=package://iti0201_robot/meshes/base_green.dae; collision sphere radius=0.005
Joints:
- removed joint camera_stand_pole_to_base
- removed joint pi_camera_to_pole

File: pibot_description/models/iti0201_robot_cone/urdf/pibot_description.urdf.xacro (robot description, xacro)
@@ -13,5 +13,19 @@
           izz="${1/2 * base_mass * (base_radius * base_radius)}"/>
       </inertial>
-      <visual name='base_visual'>
+      <visual name="base_visual">
+        <origin xyz="0.0745 -0.0725 0.0025" rpy="0 0 1.57"/>
+        <geometry>
+          <mesh filename="package://iti0201_robot/meshes/base_green.dae"/>
+          <!--cylinder length="0.0015" radius="0.07"/-->
+        </geometry>
+      </visual>
+      <collision name="base_collision">
+        <origin xyz="0.0745 -0.0725 0.0025" rpy="0 0 1.57"/>
+        <geometry>
+          <mesh filename="package://iti0201_robot/meshes/base_green.dae"/>
+          <!--cylinder length="0.0015" radius="0.07"/-->
+        </geometry>
+      </collision>
+      <!--visual name='base_visual'>
       <origin xyz="0 0 0.003" rpy="0 0 0"/>
         <geometry>
@@ -24,5 +38,5 @@
           <cylinder radius="${base_radius}" length="${base_height}"/>
         </geometry>
-      </collision>
+      </collision-->
       <visual name='front_caster_visual'>
         <origin xyz="0.035 0 0.0025" rpy="0 0 0"/>

Commit message: wheels, caster, base

File: pibot_description/models/iti0201_robot/urdf/generate_pibot.urdf.xacro (robot description, xacro)
@@ -3,12 +3,12 @@
   <xacro:include filename="$(find pibot_description)/models/iti0201_robot/urdf/pibot_description.urdf.xacro" />
   <xacro:base_with_casters/>
-  <xacro:brainbox_with_battery/>
+  <!--xacro:brainbox_with_battery/>
   <xacro:front_ir_sensors/>
   <xacro:rear_ir_sensors/>
   <xacro:first_two_line_sensors/>
   <xacro:second_two_line_sensors/>
-  <xacro:third_two_line_sensors/>
+  <xacro:third_two_line_sensors/-->
   <!--xacro:raspberry_camera/-->
   <xacro:wheels/>
-  <xacro:grabber_arm/>
+  <!--xacro:grabber_arm/-->
 </robot>

File: pibot_description/models/iti0201_robot/urdf/pibot.urdf (robot description, URDF)
Before this commit: robot pibot, 28 links, 27 joints
Links:
- removed link brainbox_with_battery
- removed link front_left_45deg_ir
- removed link front_middle_ir
- removed link front_right_45deg_ir
- removed link grabber_arm_left
- removed link grabber_arm_right
- removed link grabber_left_arm_joint
- removed link grabber_mount
- removed link grabber_pole
- removed link grabber_right_arm_joint
- removed link grabber_to_base_1
- removed link left_side_first_line_sensor_from_middle
- removed link left_side_second_line_sensor_from_middle
- removed link left_side_third_line_sensor_from_middle
- removed link pole_rotation_reference
- removed link rear_left_45deg_ir
- removed link rear_left_90deg_ir
- removed link rear_left_straight_ir
- removed link rear_right_45deg_ir
- removed link rear_right_90deg_ir
- removed link rear_right_straight_ir
- removed link right_side_first_line_sensor_from_middle
- removed link right_side_second_line_sensor_from_middle
- removed link right_side_third_line_sensor_from_middle
- link base_with_casters: geometry collision mesh filename=model://iti0201_robot/meshes/pibot2_base.dae; collision sphere radius=0.005
- link left_wheel: geometry collision cylinder length=0.009 radius=0.015; visual cylinder length=0.009 radius=0.015
- link right_wheel: geometry collision cylinder length=0.009 radius=0.015; visual cylinder length=0.009 radius=0.015
Joints:
- removed joint brainbox_to_base
- removed joint front_left_45deg_ir_to_base
- removed joint front_middle_ir_to_base
- removed joint front_right_45deg_ir_to_base
- removed joint grabber_arm_left_to_grabber_joint
- removed joint grabber_arm_right_to_grabber_joint
- removed joint grabber_left_arm_joint_to_grabber_mount
- removed joint grabber_mount_to_pole
- removed joint grabber_pole
- removed joint grabber_right_arm_joint_to_grabber_mount
- removed joint grabber_to_base_joint_1
- removed joint left_side_first_line_sensor_from_middle_to_base
- removed joint left_side_second_line_sensor_from_middle_to_base
- removed joint left_side_third_line_sensor_from_middle_to_base
- removed joint pole_rotation_reference_to_base
- removed joint rear_left_45deg_ir_to_base
- removed joint rear_left_90deg_ir_to_base
- removed joint rear_left_straight_ir_to_base
- removed joint rear_right_45deg_ir_to_base
- removed joint rear_right_90deg_ir_to_base
- removed joint rear_right_straight_ir_to_base
- removed joint right_side_first_line_sensor_from_middle_to_base
- removed joint right_side_second_line_sensor_from_middle_to_base
- removed joint right_side_third_line_sensor_from_middle_to_base
- joint Wheel_joint_to_base: origin xyz=0 0 0.0095 rpy=0 0 0 -> xyz=-0.0295 0 0.015 rpy=0 0 0

File: pibot_description/models/iti0201_robot/urdf/pibot_description.urdf.xacro (robot description, xacro)
@@ -14,19 +14,19 @@
       </inertial>
       <visual name="base_visual">
-        <origin xyz="0.0745 -0.0725 0.0025" rpy="0 0 1.57"/>
-        <geometry>
-          <mesh filename="model://iti0201_robot/meshes/base_green.dae"/>
+        <origin xyz="-0.09 0.098 0.005" rpy="0 0 -1.57"/>
+        <geometry>
+          <mesh filename="model://iti0201_robot/meshes/pibot2_base.dae"/>
           <!--cylinder length="0.0015" radius="0.07"/-->
         </geometry>
       </visual>
       <collision name="base_collision">
-        <origin xyz="0.0745 -0.0725 0.0025" rpy="0 0 1.57"/>
-        <geometry>
-          <mesh filename="model://iti0201_robot/meshes/base_green.dae"/>
+        <origin xyz="-0.09 0.098 0.005" rpy="0 0 -1.57"/>
+        <geometry>
+          <mesh filename="model://iti0201_robot/meshes/pibot2_base.dae"/>
           <!--cylinder length="0.0015" radius="0.07"/-->
         </geometry>
       </collision>
       <visual name='front_caster_visual'>
-        <origin xyz="0.035 0 0.0025" rpy="0 0 0"/>
+        <origin xyz="0.04 0 0.005" rpy="0 0 0"/>
         <geometry>
           <sphere radius="${caster_wheel_radius}"/>
@@ -34,17 +34,5 @@
       </visual>
       <collision name='front_caster_collision'>
-        <origin xyz="0.035 0 0.0025" rpy="0 0 0"/>
-        <geometry>
-          <sphere radius="${caster_wheel_radius}"/>
-        </geometry>
-      </collision>
-      <visual name='rear_caster_visual'>
-        <origin xyz="-0.035 0 0.0025" rpy="0 0 0"/>
-        <geometry>
-          <sphere radius="${caster_wheel_radius}"/>
-        </geometry>
-      </visual>
-      <collision name='rear_caster_collision'>
-        <origin xyz="-0.035 0 0.0025" rpy="0 0 0"/>
+        <origin xyz="0.04 0 0.005" rpy="0 0 0"/>
         <geometry>
           <sphere radius="${caster_wheel_radius}"/>
@@ -78,5 +66,5 @@
     </link>
     <joint type="fixed" name="Wheel_joint_to_base">
-      <origin xyz="0 0 0.0095" rpy="0 0 0" />
+      <origin xyz="-0.0295 0 0.015" rpy="0 0 0" />
       <child link="wheel_joint"/>
       <parent link="base_with_casters" />
@@ -993,5 +981,5 @@
   <xacro:macro name="wheels">
     <xacro:property name="wheel_mass" value="1" /> <!-- real: 0.005-->
-    <xacro:property name="wheel_radius" value="0.0125"/>
+    <xacro:property name="wheel_radius" value="0.015"/>
     <xacro:property name="wheel_length" value="0.009"/>
     <link name="right_wheel">
