Commit message: The whole design has been updated, line sensors were left the way they were. Base, wheels, caster and rear ir sensors were updated. Added an image of it.

File: pibot_description/models/iti0201_robot/urdf/generate_pibot.urdf.xacro (robot description, xacro)
@@ -3,12 +3,12 @@
   <xacro:include filename="$(find pibot_description)/models/iti0201_robot/urdf/pibot_description.urdf.xacro" />
   <xacro:base_with_casters/>
-  <!--xacro:brainbox_with_battery/>
+  <xacro:brainbox_with_battery/>
   <xacro:front_ir_sensors/>
   <xacro:rear_ir_sensors/>
   <xacro:first_two_line_sensors/>
   <xacro:second_two_line_sensors/>
-  <xacro:third_two_line_sensors/-->
-  <!--xacro:raspberry_camera/-->
+  <xacro:third_two_line_sensors/>
+  <xacro:raspberry_camera/>
   <xacro:wheels/>
-  <!--xacro:grabber_arm/-->
+  <xacro:grabber_arm/>
 </robot>

File: pibot_description/models/iti0201_robot/urdf/pibot.urdf (robot description, URDF)
Before this commit: robot pibot, 4 links, 3 joints
Links:
- added link brainbox_with_battery, mass 0.001; visual box size=0.0255 0.006 0.0346; visual box size=0.0255 0.006 0.0346
- added link camera_stand_pole, mass 0.001; collision cylinder length=0.0433499 radius=0.003822; visual cylinder length=0.0433499 radius=0.003822
- added link front_left_45deg_ir, mass 0.001; collision box size=0.01 0.01 0.02; visual box size=0.01 0.01 0.02
- added link front_middle_ir, mass 0.001; collision box size=0.01 0.02 0.01; visual box size=0.01 0.02 0.01
- added link front_right_45deg_ir, mass 0.001; collision box size=0.01 0.01 0.02; visual box size=0.01 0.01 0.02
- added link grabber_arm_left, mass 0.001; collision box size=.029 .003 .002; collision box size=.029 .003 .002
- added link grabber_arm_right, mass 0.001; collision box size=.029 .003 .002; collision box size=.029 .003 .002
- added link grabber_left_arm_joint, mass 0.001; collision cylinder length=.004 radius=.002; visual cylinder length=.004 radius=.002
- added link grabber_mount, mass 0.001; collision box size=.015 .042 .0057; collision box size=.035 .006 .011
- added link grabber_pole, mass 0.001; collision cylinder length=.034 radius=.006; visual cylinder length=.034 radius=.006
- added link grabber_right_arm_joint, mass 0.001; collision cylinder length=.004 radius=.002; visual cylinder length=.004 radius=.002
- added link grabber_to_base_1, mass 0.001; collision box size=.006 .034 .03455; visual box size=.006 .034 .03455
- added link left_side_first_line_sensor_from_middle, mass 0.001; collision box size=0.0015 0.0035 0.0025; visual box size=0.0015 0.0035 0.0025
- added link left_side_second_line_sensor_from_middle, mass 0.001; collision box size=0.0015 0.0035 0.0025; visual box size=0.0015 0.0035 0.0025
- added link left_side_third_line_sensor_from_middle, mass 0.001; collision box size=0.0015 0.0035 0.0025; visual box size=0.0015 0.0035 0.0025
- added link pi_camera, mass 0.001; collision box size=0.017 0.024 0.024; visual box size=0.017 0.024 0.024
- added link pole_rotation_reference, mass 0.001; collision box size=.001 .001 .001; visual box size=.001 .001 .001
- added link rear_left_45deg_ir, mass 0.001; collision box size=0.012 0.008 0.0135; visual box size=0.012 0.008 0.0135
- added link rear_left_90deg_ir, mass 0.001; collision box size=0.012 0.008 0.0135; visual box size=0.012 0.008 0.0135
- added link rear_left_straight_ir, mass 0.001; collision box size=0.012 0.008 0.0135; visual box size=0.012 0.008 0.0135
- added link rear_right_45deg_ir, mass 0.001; collision box size=0.012 0.008 0.0135; visual box size=0.012 0.008 0.0135
- added link rear_right_90deg_ir, mass 0.001; collision box size=0.012 0.008 0.0135; visual box size=0.012 0.008 0.0135
- added link rear_right_straight_ir, mass 0.001; collision box size=0.012 0.008 0.0135; visual box size=0.012 0.008 0.0135
- added link right_side_first_line_sensor_from_middle, mass 0.001; collision box size=0.0015 0.0035 0.0025; visual box size=0.0015 0.0035 0.0025
- added link right_side_second_line_sensor_from_middle, mass 0.001; collision box size=0.0015 0.0035 0.0025; visual box size=0.0015 0.0035 0.0025
- added link right_side_third_line_sensor_from_middle, mass 0.001; collision box size=0.0015 0.0035 0.0025; visual box size=0.0015 0.0035 0.0025
Joints:
- added joint brainbox_to_base: type fixed, parent base_with_casters, child brainbox_with_battery, origin xyz=0 0 0.003 rpy=0 0 0
- added joint camera_stand_pole_to_base: type fixed, parent base_with_casters, child camera_stand_pole, origin xyz=0.02940475 0 0.1135341 rpy=0 1.5707 1.5707
- added joint front_left_45deg_ir_to_base: type fixed, parent base_with_casters, child front_left_45deg_ir, origin xyz=0.0326151 0.0470558 0.016 rpy=0 0 0.78535
- added joint front_middle_ir_to_base: type fixed, parent base_with_casters, child front_middle_ir, origin xyz=0.059312 0 0.011 rpy=0 0 0
- added joint front_right_45deg_ir_to_base: type fixed, parent base_with_casters, child front_right_45deg_ir, origin xyz=0.0326 -0.0471 0.016 rpy=0 0 -0.78535
- added joint grabber_arm_left_to_grabber_joint: type fixed, parent grabber_left_arm_joint, child grabber_arm_left, origin xyz=0 0 0 rpy=0 3.1414 0
- added joint grabber_arm_right_to_grabber_joint: type fixed, parent grabber_right_arm_joint, child grabber_arm_right, origin xyz=0 0 0 rpy=0 3.1414 0
- added joint grabber_left_arm_joint_to_grabber_mount: type revolute, parent grabber_mount, child grabber_left_arm_joint, origin xyz=0.025 0.01 -0.01355 rpy=0 3.1414 0, axis 0 0 1, limit lower=0.0 upper=0.7 effort=10.0 velocity=1.0
- added joint grabber_mount_to_pole: type fixed, parent grabber_pole, child grabber_mount, origin xyz=0 0 0 rpy=1.5707 0 3.1414
- added joint grabber_pole: type revolute, parent pole_rotation_reference, child grabber_pole, origin xyz=0 0 0 rpy=0 0 0, axis 0 0 1, limit lower=0.0 upper=1.5 effort=10.0 velocity=1.0
- added joint grabber_right_arm_joint_to_grabber_mount: type revolute, parent grabber_mount, child grabber_right_arm_joint, origin xyz=0.025 -0.01 -0.01355 rpy=0 3.1414 0, axis 0 0 1, limit lower=0.0 upper=-0.7 effort=10.0 velocity=1.0
- added joint grabber_to_base_joint_1: type fixed, parent base_with_casters, child grabber_to_base_1, origin xyz=0.055 0 0.0235 rpy=0 0 0
- added joint left_side_first_line_sensor_from_middle_to_base: type fixed, parent base_with_casters, child left_side_first_line_sensor_from_middle, origin xyz=-0.0629 0.005 0.0044 rpy=0 1.5707 0
- added joint left_side_second_line_sensor_from_middle_to_base: type fixed, parent base_with_casters, child left_side_second_line_sensor_from_middle, origin xyz=-0.06289935 0.015 0.0044 rpy=0 1.5707 0
- added joint left_side_third_line_sensor_from_middle_to_base: type fixed, parent base_with_casters, child left_side_third_line_sensor_from_middle, origin xyz=-0.0541 0.035 0.0044 rpy=0 1.5707 0
- added joint pi_camera_to_pole: type fixed, parent camera_stand_pole, child pi_camera, origin xyz=0 -0.0104 0 rpy=0 0 -1.5707
- added joint pole_rotation_reference_to_base: type fixed, parent base_with_casters, child pole_rotation_reference, origin xyz=0.059 0 0.04555 rpy=0 1.5707 1.5707
- added joint rear_left_45deg_ir_to_base: type fixed, parent base_with_casters, child rear_left_45deg_ir, origin xyz=-0.0585 0.045 0.013 rpy=0 0 2.35605
- added joint rear_left_90deg_ir_to_base: type fixed, parent base_with_casters, child rear_left_90deg_ir, origin xyz=-0.05 0.058 0.013 rpy=0 0 1.5707
- added joint rear_left_straight_ir_to_base: type fixed, parent base_with_casters, child rear_left_straight_ir, origin xyz=-0.06 0.03 0.013 rpy=0 0 3.14
- added joint rear_right_45deg_ir_to_base: type fixed, parent base_with_casters, child rear_right_45deg_ir, origin xyz=-0.0585 -0.045 0.013 rpy=0 0 -2.35605
- added joint rear_right_90deg_ir_to_base: type fixed, parent base_with_casters, child rear_right_90deg_ir, origin xyz=-0.05 -0.058 0.013 rpy=0 0 -1.5707
- added joint rear_right_straight_ir_to_base: type fixed, parent base_with_casters, child rear_right_straight_ir, origin xyz=-0.06 -0.03 0.013 rpy=0 0 -3.14
- added joint right_side_first_line_sensor_from_middle_to_base: type fixed, parent base_with_casters, child right_side_first_line_sensor_from_middle, origin xyz=-0.0629 -0.005 0.0044 rpy=0 1.5707 0
- added joint right_side_second_line_sensor_from_middle_to_base: type fixed, parent base_with_casters, child right_side_second_line_sensor_from_middle, origin xyz=-0.06289935 -0.015 0.0044 rpy=0 1.5707 0
- added joint right_side_third_line_sensor_from_middle_to_base: type fixed, parent base_with_casters, child right_side_third_line_sensor_from_middle, origin xyz=-0.0541 -0.035 0.0044 rpy=0 1.5707 0
- joint Wheel_joint_to_base: origin xyz=-0.0295 0 0.015 rpy=0 0 0 -> xyz=-0.0285 0 0.015 rpy=0 0 0

File: pibot_description/models/iti0201_robot/urdf/pibot_description.urdf.xacro (robot description, xacro)
@@ -66,5 +66,5 @@
     </link>
     <joint type="fixed" name="Wheel_joint_to_base">
-      <origin xyz="-0.0295 0 0.015" rpy="0 0 0" />
+      <origin xyz="-0.0285 0 0.015" rpy="0 0 0" />
       <child link="wheel_joint"/>
       <parent link="base_with_casters" />
@@ -106,5 +106,5 @@
     </link>
     <joint type="fixed" name="brainbox_to_base">
-      <origin xyz="0 0 0" rpy="0 0 0"/>
+      <origin xyz="0 0 0.003" rpy="0 0 0"/>
       <child link="brainbox_with_battery"/>
       <parent link="base_with_casters"/>
@@ -132,5 +132,5 @@
     </link>
     <joint type="fixed" name="front_right_45deg_ir_to_base">
-      <origin xyz="0.0326 -0.0471 0.0138" rpy="0 0 -0.78535"/>
+      <origin xyz="0.0326 -0.0471 0.016" rpy="0 0 -0.78535"/>
       <child link="front_right_45deg_ir"/>
       <parent link="base_with_casters"/>
@@ -178,5 +178,5 @@
     </link>
     <joint type="fixed" name="front_middle_ir_to_base">
-      <origin xyz="0.059312 0 0.0088" rpy="0 0 0"/>
+      <origin xyz="0.059312 0 0.011" rpy="0 0 0"/>
       <child link="front_middle_ir"/>
       <parent link="base_with_casters"/>
@@ -224,5 +224,5 @@
     </link>
     <joint type="fixed" name="front_left_45deg_ir_to_base">
-      <origin xyz="0.0326151 0.0470558 0.0138" rpy="0 0 0.78535"/>
+      <origin xyz="0.0326151 0.0470558 0.016" rpy="0 0 0.78535"/>
       <child link="front_left_45deg_ir"/>
       <parent link="base_with_casters"/>
@@ -273,5 +273,5 @@
     </link>
     <joint type="fixed" name="rear_right_90deg_ir_to_base">
-      <origin xyz="-0.02256 -0.0547 0.01134" rpy="0 0 -1.5707" />
+      <origin xyz="-0.05 -0.058 0.013" rpy="0 0 -1.5707" />
       <child link="rear_right_90deg_ir"/>
       <parent link="base_with_casters"/>
@@ -319,5 +319,5 @@
     </link>
     <joint type="fixed" name="rear_right_45deg_ir_to_base">
-      <origin xyz="-0.037845 -0.046812 0.011341" rpy="0 0 -2.35605" />
+      <origin xyz="-0.0585 -0.045 0.013" rpy="0 0 -2.35605" />
       <child link="rear_right_45deg_ir"/>
       <parent link="base_with_casters"/>
@@ -365,5 +365,5 @@
     </link>
     <joint type="fixed" name="rear_right_straight_ir_to_base">
-      <origin xyz="-0.0501109 -0.035473 0.011341" rpy="0 0 -3.14" />
+      <origin xyz="-0.06 -0.03 0.013" rpy="0 0 -3.14" />
       <child link="rear_right_straight_ir"/>
       <parent link="base_with_casters"/>
@@ -411,5 +411,5 @@
     </link>
     <joint type="fixed" name="rear_left_90deg_ir_to_base">
-      <origin xyz="-0.0225688 0.054749 0.011341" rpy="0 0 1.5707" />
+      <origin xyz="-0.05 0.058 0.013" rpy="0 0 1.5707" />
       <child link="rear_left_90deg_ir"/>
       <parent link="base_with_casters"/>
@@ -457,5 +457,5 @@
     </link>
     <joint type="fixed" name="rear_left_45deg_ir_to_base">
-      <origin xyz="-0.037845 0.046812 0.011341" rpy="0 0 2.35605" />
+      <origin xyz="-0.0585 0.045 0.013" rpy="0 0 2.35605" />
       <child link="rear_left_45deg_ir"/>
       <parent link="base_with_casters"/>
@@ -503,5 +503,5 @@
     </link>
     <joint type="fixed" name="rear_left_straight_ir_to_base">
-      <origin xyz="-0.0501109 0.035473 0.011341" rpy="0 0 3.14" />
+      <origin xyz="-0.06 0.03 0.013" rpy="0 0 3.14" />
       <child link="rear_left_straight_ir"/>
       <parent link="base_with_casters"/>
@@ -553,5 +553,5 @@
     </link>
     <joint type="fixed" name="right_side_first_line_sensor_from_middle_to_base">
-      <origin xyz="-0.0629 -0.005 0.0014545" rpy="0 1.5707 0" />
+      <origin xyz="-0.0629 -0.005 0.0044" rpy="0 1.5707 0" />
       <child link="right_side_first_line_sensor_from_middle"/>
       <parent link="base_with_casters"/>
@@ -610,5 +610,5 @@
     </link>
     <joint type="fixed" name="left_side_first_line_sensor_from_middle_to_base">
-      <origin xyz="-0.0629 0.005 0.0014545" rpy="0 1.5707 0" />
+      <origin xyz="-0.0629 0.005 0.0044" rpy="0 1.5707 0" />
       <child link="left_side_first_line_sensor_from_middle"/>
       <parent link="base_with_casters"/>
@@ -670,5 +670,5 @@
     </link>
     <joint type="fixed" name="right_side_second_line_sensor_from_middle_to_base">
-      <origin xyz="-0.06289935 -0.015 0.0014545" rpy="0 1.5707 0" />
+      <origin xyz="-0.06289935 -0.015 0.0044" rpy="0 1.5707 0" />
       <child link="right_side_second_line_sensor_from_middle"/>
       <parent link="base_with_casters"/>
@@ -728,5 +728,5 @@
     </link>
     <joint type="fixed" name="left_side_second_line_sensor_from_middle_to_base">
-      <origin xyz="-0.06289935 0.015 0.0014545" rpy="0 1.5707 0" />
+      <origin xyz="-0.06289935 0.015 0.0044" rpy="0 1.5707 0" />
       <child link="left_side_second_line_sensor_from_middle"/>
       <parent link="base_with_casters"/>
@@ -788,5 +788,5 @@
     </link>
     <joint type="fixed" name="right_side_third_line_sensor_from_middle_to_base">
-      <origin xyz="-0.0541 -0.035 0.0014545" rpy="0 1.5707 0" />
+      <origin xyz="-0.0541 -0.035 0.0044" rpy="0 1.5707 0" />
       <child link="right_side_third_line_sensor_from_middle"/>
       <parent link="base_with_casters"/>
@@ -846,5 +846,5 @@
     </link>
     <joint type="fixed" name="left_side_third_line_sensor_from_middle_to_base">
-      <origin xyz="-0.0541 0.035 0.0014545" rpy="0 1.5707 0" />
+      <origin xyz="-0.0541 0.035 0.0044" rpy="0 1.5707 0" />
       <child link="left_side_third_line_sensor_from_middle"/>
       <parent link="base_with_casters"/>

Commit message: Added script to kill gazebo if it is running before the start of test.

File: pibot_description/models/iti0201_robot/urdf/generate_pibot.urdf.xacro (robot description, xacro)
@@ -2,4 +2,32 @@
 <robot xmlns:xacro="http://www.ros.org/wiki/xacro" name="pibot">
   <xacro:include filename="$(find pibot_description)/models/iti0201_robot/urdf/pibot_description.urdf.xacro" />
+  <xacro:property name="camera_link" value="0.05" /> <!-- Size of square 'camera' box -->
+  <joint name="camera_joint" type="fixed">
+    <axis xyz="0 1 0" />
+    <origin xyz="${camera_link} 0 1" rpy="0 0 0"/>
+    <parent link="base_with_casters"/>
+    <child link="camera_link"/>
+  </joint>
+  <!-- Camera -->
+  <link name="camera_link">
+    <collision>
+      <origin xyz="0 0 0" rpy="0 0 0"/>
+      <geometry>
+    <box size="${camera_link} ${camera_link} ${camera_link}"/>
+      </geometry>
+    </collision>
+    <visual>
+      <origin xyz="0 0 0" rpy="0 0 0"/>
+      <geometry>
+    <box size="${camera_link} ${camera_link} ${camera_link}"/>
+      </geometry>
+      <material name="red"/>
+    </visual>
+    <inertial>
+      <mass value="1e-5" />
+      <origin xyz="0 0 0" rpy="0 0 0"/>
+      <inertia ixx="1e-6" ixy="0" ixz="0" iyy="1e-6" iyz="0" izz="1e-6" />
+    </inertial>
+  </link>
   <xacro:base_with_casters/>
   <xacro:brainbox_with_battery/>

Commit message: Removed camera visualization

File: pibot_description/models/iti0201_robot/urdf/generate_pibot.urdf.xacro (robot description, xacro)
@@ -2,32 +2,4 @@
 <robot xmlns:xacro="http://www.ros.org/wiki/xacro" name="pibot">
   <xacro:include filename="$(find pibot_description)/models/iti0201_robot/urdf/pibot_description.urdf.xacro" />
-  <xacro:property name="camera_link" value="0.05" /> <!-- Size of square 'camera' box -->
-  <joint name="camera_joint" type="fixed">
-    <axis xyz="0 1 0" />
-    <origin xyz="${camera_link} 0 1" rpy="0 0 0"/>
-    <parent link="base_with_casters"/>
-    <child link="camera_link"/>
-  </joint>
-  <!-- Camera -->
-  <link name="camera_link">
-    <collision>
-      <origin xyz="0 0 0" rpy="0 0 0"/>
-      <geometry>
-    <box size="${camera_link} ${camera_link} ${camera_link}"/>
-      </geometry>
-    </collision>
-    <visual>
-      <origin xyz="0 0 0" rpy="0 0 0"/>
-      <geometry>
-    <box size="${camera_link} ${camera_link} ${camera_link}"/>
-      </geometry>
-      <material name="red"/>
-    </visual>
-    <inertial>
-      <mass value="1e-5" />
-      <origin xyz="0 0 0" rpy="0 0 0"/>
-      <inertia ixx="1e-6" ixy="0" ixz="0" iyy="1e-6" iyz="0" izz="1e-6" />
-    </inertial>
-  </link>
   <xacro:base_with_casters/>
   <xacro:brainbox_with_battery/>
